File: Hardware/KeyBoard/KeyBoard.kicad_pcb (KiCad board)
At the start: 2 copper layers, 319.1 x 128.7 mm, 243 parts, among them X1 8MHz

Commit message: complete layout
Parts:
- removed LED100, LED101, LED83, LED84, LED85, LED86, LED87, LED88, LED89, LED90, LED91, LED92, LED93, LED94, LED95, LED96, LED97, LED98, LED99: ~, persional_library:LED-SMD_L3.2-W2.8_YO-WS2812B-3528
- removed SW1: ~, persional_library:SW-SMD_L6.0-W3.3-LS8.0
- added C14: 10uF, persional_library:C0402, B.Cu at (594.0, 14.5)
- added C15: 100nF, persional_library:C0402, B.Cu at (595.2, 14.5)
- added C16: 10uF, persional_library:C0402, B.Cu at (603.8, 11.9)
- added C17: 100nF, persional_library:C0402, B.Cu at (344.5, 4.36)
- added C18: 10uF, persional_library:C0402, B.Cu at (343.2, 4.36)
- added C19: 100nF, persional_library:C0402, B.Cu at (343.1, 14.4)
- added C20: 10uF, persional_library:C0402, B.Cu at (341.2, 13.9)
- added D1: ~, persional_library:SOD-523_L1.2-W0.8-LS1.6-FD, B.Cu at (332.1, 13.9)
- added FPC4: ~, persional_library:FPC-SMD_P0.50-8P_FGS-XJ-H2.0, B.Cu at (426.6, 6.42)
- added Q1: ~, persional_library:POWERTDFN-8_L3.1-W3.1-P0.65-LS3.3-BL, B.Cu at (329.1, 15.8)
- added Q2: ~, persional_library:SOT-23-3_L2.9-W1.3-P1.90-LS2.4-BR, B.Cu at (334.5, 16.8)
- added R28: 10KΩ, persional_library:R0402, B.Cu at (601.4, 32.5)
- added R29: 10KΩ, persional_library:R0402, B.Cu at (599.1, 44.0)
- added R30: 5.1kΩ, persional_library:R0402, B.Cu at (601.6, 11.3)
- added R31: 5.1kΩ, persional_library:R0402, B.Cu at (598.6, 11.3)
- added R32: 100kΩ, persional_library:R0402, B.Cu at (596.5, 14.4)
- added R33: 4.7Ω, persional_library:R0402, B.Cu at (603.7, 13.2)
- added R34: 10kΩ, persional_library:R0402, B.Cu at (335.1, 14.5)
- added R35: 10kΩ, persional_library:R0402, B.Cu at (335.1, 13.3)
- added R36: 100kΩ, persional_library:R0402, B.Cu at (332.1, 16.3)
- added R37: 1kΩ, persional_library:R0402, B.Cu at (340.0, 5.10)
- added U15: ~, persional_library:SOP-16, B.Cu at (602.6, 17.8)
- added U16: ~, persional_library:CONN-SMD_2P-P2.50_HCTL_HC-XH-2ALT, B.Cu at (331.8, 7.10)
- added U17: ~, persional_library:ESOP-8_L4.9-W3.9-P1.27-LS6.0-BL-EP, B.Cu at (341.2, 9.40)
- added USBC1: ~, persional_library:USB-C-SMD_TYPE-C-USB-17, B.Cu at (599.9, 6.70)
- C1, C10, C11, C12, C13, C2, C3, C4, C5, C6, C7, C8, C9, CN1, FPC1, FPC2, FPC3, KEY1, KEY10, KEY11, KEY12, KEY13, KEY14, KEY15, KEY16, KEY17, KEY18, KEY19, KEY2, KEY20, KEY21, KEY22, KEY23, KEY24, KEY25, KEY26, KEY27, KEY28, KEY29, KEY3, KEY30, KEY31, KEY32, KEY33, KEY34, KEY35, KEY36, KEY37, KEY38, KEY39, KEY4, KEY40, KEY41, KEY42, KEY43, KEY44, KEY45, KEY46, KEY47, KEY48, KEY49, KEY5, KEY50, KEY51, KEY52, KEY53, KEY54, KEY55, KEY56, KEY57, KEY58, KEY59, KEY6, KEY60, KEY61, KEY62, KEY63, KEY64, KEY65, KEY66, KEY67, KEY68, KEY69, KEY7, KEY70, KEY71, KEY72, KEY73, KEY74, KEY75, KEY76, KEY77, KEY78, KEY79, KEY8, KEY80, KEY81, KEY82, KEY9, LED1, LED10, LED11, LED12, LED13, LED14, LED15, LED16, LED17, LED18, LED19, LED2, LED20, LED21, LED22, LED23, LED24, LED25, LED26, LED27, LED28, LED29, LED3, LED30, LED31, LED32, LED33, LED34, LED35, LED36, LED37, LED38, LED39, LED4, LED40, LED41, LED42, LED43, LED44, LED45, LED46, LED47, LED48, LED49, LED5, LED50, LED51, LED52, LED53, LED54, LED55, LED56, LED57, LED58, LED59, LED6, LED60, LED61, LED62, LED63, LED64, LED65, LED66, LED67, LED68, LED69, LED7, LED70, LED71, LED72, LED73, LED74, LED75, LED76, LED77, LED78, LED79, LED8, LED80, LED81, LED82, LED9, R1, R10, R11, R12, R13, R14, R15, R16, R17, R18, R19, R2, R20, R21, R22, R23, R24, R25, R26, R27, R3, R4, R5, R6, R7, R8, R9, U1, U10, U11, U12, U13, U14, U2, U3, U4, U5, U6, U7, U8, U9, X1: moved to B.Cu
- moved LED14 573.9 mm to (616.9, 6.19)
- moved LED15 564.3 mm to (616.9, 46.7), turned to 180 degrees
- moved LED44 543.4 mm to (616.9, 65.7)
- moved LED13 540.8 mm to (583.6, 6.08)
- moved LED45 540.6 mm to (616.9, 84.6), turned to 180 degrees
- moved LED12 521.3 mm to (564.5, 6.08)
- moved LED72 519.8 mm to (616.9, 103.8)
- moved LED73 513.1 mm to (612.1, 127.6), turned to 180 degrees
- moved LED43 505.2 mm to (578.8, 65.7)
- moved LED16 502.5 mm to (574.0, 46.5), turned to 180 degrees
- moved LED11 501.8 mm to (545.5, 6.19)
- moved LED71 495.1 mm to (593.1, 108.7)
- moved LED74 494.5 mm to (593.1, 127.6), turned to 180 degrees
- moved X1 492.4 mm to (607.5, 36.8), turned to -90 degrees
- moved CN1 489.9 mm to (623.0, 25.0), turned to -90 degrees
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Connections:
- FPC2 pad 1: /MCU/UART_RX -> /Device/USB_DM_2
- FPC2 pad 2: /MCU/UART_TX -> /Device/USB_DP_2
- FPC2 pad 3: /MCU/USB_PORT_P -> /MCU/UART_TX
- FPC2 pad 4: /MCU/USB_PORT_N -> /MCU/UART_RX
- KEY1 pad 2: Net-(U1-D5) -> Net-(U1-D7)
- KEY2 pad 2: Net-(U1-D1) -> Net-(U1-D6)
- KEY25 pad 2: Net-(U4-D4) -> Net-(U4-D7)
- KEY26 pad 2: Net-(U4-D4) -> Net-(U4-D6)
- KEY27 pad 2: Net-(U4-D4) -> Net-(U4-D5)
- KEY29 pad 2: Net-(U4-D0) -> Net-(U4-D3)
- KEY30 pad 2: Net-(U4-D0) -> Net-(U4-D2)
- KEY31 pad 2: Net-(U4-D0) -> Net-(U4-D1)
- KEY4 pad 2: Net-(U1-D1) -> Net-(U1-D4)
- KEY5 pad 2: Net-(U1-D1) -> Net-(U1-D3)
- KEY6 pad 2: Net-(U1-D0) -> Net-(U1-D2)
- LED82 pad 2: Net-(LED82-DOUT) -> unconnected-(LED82-DOUT-Pad2)
- R1 pad 1: +3V3 -> Net-(U1-D7)
- R1 pad 2: +3V3 -> Net-(U1-D6)
- R1 pad 3: +3V3 -> Net-(U1-D5)
- R1 pad 4: +3V3 -> Net-(U1-D4)
- R1 pad 5: Net-(U1-D1) -> +3V3
- R1 pad 6: Net-(U1-D5) -> +3V3
- R1 pad 7: Net-(U1-D1) -> +3V3
- R1 pad 8: Net-(U1-D5) -> +3V3
- R10 pad 1: +3V3 -> Net-(U5-D3)
- R10 pad 2: +3V3 -> Net-(U5-D2)
- R10 pad 3: +3V3 -> Net-(U5-D1)
- R10 pad 4: +3V3 -> Net-(U5-D0)
- R10 pad 5: Net-(U5-D0) -> +3V3
- R10 pad 6: Net-(U5-D1) -> +3V3
- R10 pad 7: Net-(U5-D2) -> +3V3
- R10 pad 8: Net-(U5-D3) -> +3V3
- R11 pad 1: +3V3 -> Net-(U6-D7)
- R11 pad 2: +3V3 -> Net-(U6-D6)
- R11 pad 3: +3V3 -> Net-(U6-D5)
- R11 pad 4: +3V3 -> Net-(U6-D4)
- R11 pad 5: Net-(U6-D4) -> +3V3
- R11 pad 6: Net-(U6-D5) -> +3V3
- R11 pad 7: Net-(U6-D6) -> +3V3
- R11 pad 8: Net-(U6-D7) -> +3V3
- R12 pad 1: +3V3 -> Net-(U6-D3)
- R12 pad 2: +3V3 -> Net-(U6-D2)
- R12 pad 3: +3V3 -> Net-(U6-D1)
- R12 pad 4: +3V3 -> Net-(U6-D0)
- R12 pad 5: Net-(U6-D0) -> +3V3
- R12 pad 6: Net-(U6-D1) -> +3V3
- R12 pad 7: Net-(U6-D2) -> +3V3
- R12 pad 8: Net-(U6-D3) -> +3V3
- R13 pad 1: +3V3 -> Net-(U7-D7)
- R13 pad 2: +3V3 -> Net-(U7-D6)
- R13 pad 3: +3V3 -> Net-(U7-D5)
- R13 pad 4: +3V3 -> Net-(U7-D4)
- R13 pad 5: Net-(U7-D4) -> +3V3
- R13 pad 6: Net-(U7-D5) -> +3V3
- R13 pad 7: Net-(U7-D6) -> +3V3
- R13 pad 8: Net-(U7-D7) -> +3V3
- R14 pad 1: +3V3 -> Net-(U7-D3)
- R14 pad 2: +3V3 -> Net-(U7-D2)
- R14 pad 3: +3V3 -> Net-(U7-D1)
- R14 pad 4: +3V3 -> Net-(U7-D0)
- R14 pad 5: Net-(U7-D0) -> +3V3
- R14 pad 6: Net-(U7-D1) -> +3V3
- R14 pad 7: Net-(U7-D2) -> +3V3
- R14 pad 8: Net-(U7-D3) -> +3V3
- R15 pad 1: +3V3 -> Net-(U8-D7)
- R15 pad 2: +3V3 -> Net-(U8-D6)
- R15 pad 3: +3V3 -> Net-(U8-D5)
- R15 pad 4: +3V3 -> Net-(U8-D4)
- R15 pad 5: Net-(U8-D4) -> +3V3
- R15 pad 6: Net-(U8-D5) -> +3V3
- R15 pad 7: Net-(U8-D6) -> +3V3
- R15 pad 8: Net-(U8-D7) -> +3V3
- R16 pad 1: +3V3 -> Net-(U8-D3)
- R16 pad 2: +3V3 -> Net-(U8-D2)
- R16 pad 3: +3V3 -> Net-(U8-D1)
- R16 pad 4: +3V3 -> Net-(U8-D0)
- R16 pad 5: Net-(U8-D0) -> +3V3
- R16 pad 6: Net-(U8-D1) -> +3V3
- R16 pad 7: Net-(U8-D2) -> +3V3
- R16 pad 8: Net-(U8-D3) -> +3V3
- R17 pad 1: +3V3 -> Net-(U9-D7)
- R17 pad 2: +3V3 -> Net-(U9-D6)
- R17 pad 3: +3V3 -> Net-(U9-D5)
- R17 pad 4: +3V3 -> Net-(U9-D4)
- R17 pad 5: Net-(U9-D4) -> +3V3
- R17 pad 6: Net-(U9-D5) -> +3V3
- R17 pad 7: Net-(U9-D6) -> +3V3
- R17 pad 8: Net-(U9-D7) -> +3V3
- R18 pad 1: +3V3 -> Net-(U9-D3)
- R18 pad 2: +3V3 -> Net-(U9-D2)
- R18 pad 3: +3V3 -> Net-(U9-D1)
- R18 pad 4: +3V3 -> Net-(U9-D0)
- R18 pad 5: Net-(U9-D0) -> +3V3
- R18 pad 6: Net-(U9-D1) -> +3V3
- R18 pad 7: Net-(U9-D2) -> +3V3
- R18 pad 8: Net-(U9-D3) -> +3V3
- R19 pad 1: +3V3 -> Net-(U10-D7)
- R19 pad 2: +3V3 -> Net-(U10-D6)
- R19 pad 3: +3V3 -> Net-(U10-D5)
- R19 pad 4: +3V3 -> Net-(U10-D4)
- R19 pad 5: Net-(U10-D4) -> +3V3
- R19 pad 6: Net-(U10-D5) -> +3V3
- R19 pad 7: Net-(U10-D6) -> +3V3
- R19 pad 8: Net-(U10-D7) -> +3V3
- R2 pad 1: +3V3 -> Net-(U1-D3)
- R2 pad 2: +3V3 -> Net-(U1-D2)
- R2 pad 3: +3V3 -> Net-(U1-D1)
- R2 pad 4: +3V3 -> Net-(U1-D0)
- R2 pad 5: Net-(U1-D0) -> +3V3
- R2 pad 6: Net-(U1-D1) -> +3V3
- R2 pad 7: Net-(U1-D0) -> +3V3
- R2 pad 8: Net-(U1-D1) -> +3V3
- R20 pad 1: +3V3 -> Net-(U10-D3)
- R20 pad 2: +3V3 -> Net-(U10-D2)
- R20 pad 3: +3V3 -> Net-(U10-D1)
- R20 pad 4: +3V3 -> Net-(U10-D0)
- R20 pad 5: Net-(U10-D0) -> +3V3
- R20 pad 6: Net-(U10-D1) -> +3V3
- R20 pad 7: Net-(U10-D2) -> +3V3
- R20 pad 8: Net-(U10-D3) -> +3V3
- R21 pad 1: +3V3 -> Net-(U11-D7)
- R21 pad 2: +3V3 -> Net-(U11-D6)
- R21 pad 3: +3V3 -> Net-(U11-D5)
- R21 pad 4: +3V3 -> Net-(U11-D4)
- R21 pad 5: Net-(U11-D4) -> +3V3
- R21 pad 6: Net-(U11-D5) -> +3V3
- R21 pad 7: Net-(U11-D6) -> +3V3
- R21 pad 8: Net-(U11-D7) -> +3V3
- R22 pad 1: +3V3 -> Net-(U11-D3)
- R22 pad 2: +3V3 -> Net-(U11-D2)
- R22 pad 3: +3V3 -> Net-(U11-D1)
- R22 pad 4: +3V3 -> Net-(U11-D0)
- R22 pad 5: Net-(U11-D0) -> +3V3
- R22 pad 6: Net-(U11-D1) -> +3V3
- R22 pad 7: Net-(U11-D2) -> +3V3
- R22 pad 8: Net-(U11-D3) -> +3V3
- R25 pad 2: /MCU/USB_PORT_N -> /Device/USB_DM_1
- R26 pad 2: /MCU/USB_PORT_P -> /Device/USB_DP_1
- R27 pad 1: /MCU/USB_PORT_P -> /Device/USB_DP_1
- R3 pad 1: +3V3 -> Net-(U2-D7)
- R3 pad 2: +3V3 -> Net-(U2-D6)
- R3 pad 3: +3V3 -> Net-(U2-D5)
- R3 pad 4: +3V3 -> Net-(U2-D4)
- R3 pad 5: Net-(U2-D4) -> +3V3
- R3 pad 6: Net-(U2-D5) -> +3V3
- R3 pad 7: Net-(U2-D6) -> +3V3
- R3 pad 8: Net-(U2-D7) -> +3V3
- R4 pad 1: +3V3 -> Net-(U2-D3)
- R4 pad 2: +3V3 -> Net-(U2-D2)
- R4 pad 3: +3V3 -> Net-(U2-D1)
- R4 pad 4: +3V3 -> Net-(U2-D0)
- R4 pad 5: Net-(U2-D0) -> +3V3
- R4 pad 6: Net-(U2-D1) -> +3V3
- R4 pad 7: Net-(U2-D2) -> +3V3
- R4 pad 8: Net-(U2-D3) -> +3V3
- R5 pad 1: +3V3 -> Net-(U3-D7)
- R5 pad 2: +3V3 -> Net-(U3-D6)
- R5 pad 3: +3V3 -> Net-(U3-D5)
- R5 pad 4: +3V3 -> Net-(U3-D4)
- R5 pad 5: Net-(U3-D4) -> +3V3
- R5 pad 6: Net-(U3-D5) -> +3V3
- R5 pad 7: Net-(U3-D6) -> +3V3
- R5 pad 8: Net-(U3-D7) -> +3V3
- R6 pad 1: +3V3 -> Net-(U3-D3)
- R6 pad 2: +3V3 -> Net-(U3-D2)
- R6 pad 3: +3V3 -> Net-(U3-D1)
- R6 pad 4: +3V3 -> Net-(U3-D0)
- R6 pad 5: Net-(U3-D0) -> +3V3
- R6 pad 6: Net-(U3-D1) -> +3V3
- R6 pad 7: Net-(U3-D2) -> +3V3
- R6 pad 8: Net-(U3-D3) -> +3V3
- R7 pad 1: +3V3 -> Net-(U4-D7)
- R7 pad 2: +3V3 -> Net-(U4-D6)
- R7 pad 3: +3V3 -> Net-(U4-D5)
- R7 pad 4: +3V3 -> Net-(U4-D4)
- R7 pad 5: Net-(U4-D4) -> +3V3
- R7 pad 6: Net-(U4-D4) -> +3V3
- R7 pad 7: Net-(U4-D4) -> +3V3
- R7 pad 8: Net-(U4-D4) -> +3V3
- R8 pad 1: +3V3 -> Net-(U4-D3)
- R8 pad 2: +3V3 -> Net-(U4-D2)
- R8 pad 3: +3V3 -> Net-(U4-D1)
- R8 pad 4: +3V3 -> Net-(U4-D0)
- R8 pad 5: Net-(U4-D0) -> +3V3
- R8 pad 6: Net-(U4-D0) -> +3V3
- R8 pad 7: Net-(U4-D0) -> +3V3
- R8 pad 8: Net-(U4-D0) -> +3V3
- R9 pad 1: +3V3 -> Net-(U5-D7)
- R9 pad 2: +3V3 -> Net-(U5-D6)
- R9 pad 3: +3V3 -> Net-(U5-D5)
- R9 pad 4: +3V3 -> Net-(U5-D4)
- R9 pad 5: Net-(U5-D4) -> +3V3
- R9 pad 6: Net-(U5-D5) -> +3V3
- R9 pad 7: Net-(U5-D6) -> +3V3
- R9 pad 8: Net-(U5-D7) -> +3V3
- U1 pad 13: Net-(U1-D0) -> Net-(U1-D2)
- U1 pad 14: Net-(U1-D1) -> Net-(U1-D3)
- U1 pad 3: Net-(U1-D1) -> Net-(U1-D4)
- U1 pad 5: Net-(U1-D1) -> Net-(U1-D6)
- U1 pad 6: Net-(U1-D5) -> Net-(U1-D7)
- U13 pad 20: unconnected-(U13-PB2BOOT1-Pad20) -> Net-(U13-PB2BOOT1)
- U13 pad 44: GND -> Net-(U13-BOOT0)
- U4 pad 12: Net-(U4-D0) -> Net-(U4-D1)
- U4 pad 13: Net-(U4-D0) -> Net-(U4-D2)
- U4 pad 14: Net-(U4-D0) -> Net-(U4-D3)
- U4 pad 4: Net-(U4-D4) -> Net-(U4-D5)
- U4 pad 5: Net-(U4-D4) -> Net-(U4-D6)
- U4 pad 6: Net-(U4-D4) -> Net-(U4-D7)

Commit message: start generic cabling
Parts:
- moved R27 4.80 mm to (595.3, 29.5)
- moved R26 2.40 mm to (594.1, 29.5)
Connections:
- CN1 pad 1: /MCU/SWCLK -> /MCU/SWDIO
- CN1 pad 2: /MCU/SWDIO -> /MCU/SWCLK
Routing:
- net Net-(U1-D7): track 0.00 -> 251.0 mm, vias 0 -> 2
- net Net-(U1-D6): track 0.00 -> 211.3 mm, vias 0 -> 2
- net Net-(U2-D1): track 0.00 -> 197.8 mm
- net Net-(U1-D5): track 0.00 -> 191.6 mm, vias 0 -> 2
- net Net-(U2-D7): track 0.00 -> 178.8 mm, vias 0 -> 2
- net Net-(U2-D0): track 0.00 -> 177.2 mm, vias 0 -> 2
- net Net-(U1-D4): track 0.00 -> 172.0 mm, vias 0 -> 2
- net Net-(U2-D6): track 0.00 -> 154.8 mm, vias 0 -> 2
- net Net-(U2-D5): track 0.00 -> 140.0 mm, vias 0 -> 2
- net Net-(U1-D3): track 0.00 -> 130.0 mm
- net Net-(U2-D2): track 0.00 -> 126.0 mm
- net Net-(U2-D4): track 0.00 -> 125.3 mm, vias 0 -> 2
- net Net-(U1-D2): track 0.00 -> 103.2 mm
- net Net-(U2-D3): track 0.00 -> 94.3 mm
- net Net-(U1-D1): track 0.00 -> 86.0 mm
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
Commit message: Update the PCB layout
Parts:
- moved KEY1 307.4 mm to (616.9, 78.7), turned to 180 degrees
- moved KEY81 283.6 mm to (335.9, 40.6)
- moved KEY82 274.1 mm to (345.4, 59.7)
- moved KEY2 266.2 mm to (616.9, 59.7), turned to 180 degrees
- moved KEY3 244.6 mm to (616.9, 40.6), turned to 180 degrees
- moved KEY67 241.3 mm to (319.2, 116.8)
- moved KEY17 224.6 mm to (578.8, 59.7)
- moved KEY4 223.8 mm to (616.9, 12.1)
- moved KEY5 222.0 mm to (616.9, 97.8), turned to 180 degrees
- moved KEY15 209.5 mm to (526.4, 40.6)
- moved KEY6 203.5 mm to (612.1, 121.6), turned to 180 degrees
- moved KEY66 189.1 mm to (343.1, 116.8)
- moved KEY72 187.3 mm to (324.0, 78.7)
- moved KEY55 183.4 mm to (388.3, 78.7)
- moved KEY18 182.0 mm to (555.0, 59.7)
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Connections:
- net /Device/USB_DM_1 renamed /Device/USB_1_DN
- net /Device/USB_DM_2 renamed /Device/USB_2_DN
- net /Device/USB_DM_3 renamed /Device/USB_3_DN
- net /Device/USB_DM_4 renamed /Device/USB_4_DN
- net /Device/USB_DM_HUB renamed /Device/USB_HUB_DN
- net /Device/USB_DP_1 renamed /Device/USB_1_DP
- net /Device/USB_DP_2 renamed /Device/USB_2_DP
- net /Device/USB_DP_3 renamed /Device/USB_3_DP
- net /Device/USB_DP_4 renamed /Device/USB_4_DP
- net /Device/USB_DP_HUB renamed /Device/USB_HUB_DP
Routing:
- net Net-(U1-D7): track 251.0 -> 2.64 mm, vias 2 -> 0
- net Net-(U1-D6): track 211.3 -> 2.44 mm, vias 2 -> 0
- net Net-(U1-D5): track 191.6 -> 2.44 mm, vias 2 -> 0
- net Net-(U1-D4): track 172.0 -> 2.64 mm, vias 2 -> 0
- net Net-(U2-D1): track 197.8 -> 36.4 mm
- net Net-(U2-D0): track 177.2 -> 16.7 mm, vias 2 -> 0
- net Net-(U2-D7): track 178.8 -> 26.6 mm, vias 2 -> 0
- net Net-(U1-D0): track 69.2 -> 200.4 mm
- net Net-(U2-D6): track 154.8 -> 43.6 mm, vias 2 -> 0
- net Net-(U1-D1): track 86.0 -> 182.7 mm
- net Net-(U1-D2): track 103.2 -> 186.5 mm
- net Net-(U2-D5): track 140.0 -> 60.8 mm, vias 2 -> 0
- net Net-(LED79-DOUT): track 78.9 -> 0.00 mm
- net Net-(U2-D2): track 126.0 -> 56.9 mm
- net Net-(LED78-DOUT): track 64.1 -> 0.00 mm
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
Commit message: complete Key line
Parts:
- moved KEY69 116.1 mm to (366.9, 116.8), turned to 180 degrees
- moved KEY80 86.9 mm to (507.4, 116.8)
- moved KEY68 86.5 mm to (316.9, 12.1), turned to 0 degrees
- moved KEY70 80.6 mm to (343.1, 116.8)
- moved KEY67 76.2 mm to (316.9, 40.6)
- moved KEY77 62.1 mm to (593.1, 102.6)
- moved KEY49 61.9 mm to (416.9, 97.8)
- moved KEY57 61.9 mm to (378.8, 97.8)
- moved KEY66 61.0 mm to (321.6, 59.7)
- moved KEY29 57.3 mm to (488.3, 40.6)
- moved KEY41 57.3 mm to (435.9, 97.8)
- moved KEY44 57.3 mm to (431.2, 40.6)
- moved KEY56 57.3 mm to (393.1, 40.6)
- moved KEY64 57.3 mm to (355.0, 40.6)
- moved KEY65 57.3 mm to (324.0, 78.7)
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Routing:
- net Net-(U10-D7): track 2.64 -> 481.4 mm, vias 0 -> 2
- net Net-(U10-D0): track 2.66 -> 412.5 mm, vias 0 -> 2
- net Net-(U10-D1): track 2.46 -> 393.8 mm, vias 0 -> 2
- net Net-(U10-D4): track 2.64 -> 380.6 mm, vias 0 -> 2
- net Net-(U10-D2): track 2.46 -> 374.6 mm, vias 0 -> 2
- net Net-(U10-D5): track 2.44 -> 364.8 mm, vias 0 -> 2
- net Net-(U10-D6): track 2.44 -> 339.1 mm, vias 0 -> 2
- net Net-(U10-D3): track 2.66 -> 320.0 mm, vias 0 -> 2
- net Net-(U11-D4): track 2.66 -> 198.9 mm, vias 0 -> 2
- net Net-(U11-D3): track 2.66 -> 198.6 mm, vias 0 -> 2
- net Net-(U11-D5): track 2.46 -> 198.2 mm, vias 0 -> 2
- net Net-(U11-D2): track 2.46 -> 195.5 mm, vias 0 -> 2
- net Net-(U11-D1): track 2.46 -> 192.6 mm, vias 0 -> 2
- net Net-(U11-D0): track 2.66 -> 190.8 mm, vias 0 -> 2
- net Net-(U9-D3): track 2.66 -> 185.7 mm
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
Commit message: Complete the non-power line routing
Parts:
- moved FPC3 251.9 mm to (563.2, 25.2)
- moved FPC4 152.6 mm to (578.0, 25.2), turned to -90 degrees
- moved LED11 0.12 mm to (545.5, 6.08)
Connections:
- FPC2 pad 3: /MCU/UART_TX -> /MCU/UART_RX
- FPC2 pad 4: /MCU/UART_RX -> /MCU/UART_TX
Routing:
- net /LED/LED_CE: track 0.00 -> 337.3 mm, vias 0 -> 4
- net /KEY/SPI1_CLK: track 0.00 -> 283.3 mm, vias 0 -> 17
- net /KEY/CE: track 0.00 -> 278.7 mm, vias 0 -> 16
- net /KEY/PL: track 0.00 -> 272.4 mm, vias 0 -> 17
- net /MCU/UART_TX: track 0.00 -> 111.9 mm, vias 0 -> 2
- net /MCU/UART_RX: track 0.00 -> 110.9 mm, vias 0 -> 2
- net /Device/USB_2_DP: track 0.00 -> 104.9 mm
- net /Device/USB_2_DN: track 0.00 -> 104.9 mm
- net /KEY/SPI1_MISO: track 0.00 -> 93.4 mm, vias 0 -> 2
- net Net-(LED79-DOUT): track 0.00 -> 67.2 mm, vias 0 -> 2
- net Net-(LED78-DOUT): track 0.00 -> 64.7 mm
- net /MCU/I2C2_SCL: track 0.00 -> 50.8 mm, vias 0 -> 2
- net /MCU/I2C2_SDA: track 0.00 -> 49.8 mm, vias 0 -> 2
- net Net-(LED58-DOUT): track 0.00 -> 49.7 mm
- net /MCU/I2C1_SDA: track 0.00 -> 46.3 mm, vias 0 -> 2
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