File: Hardware/KeyBoard/LED.kicad_sch (KiCad schematic)
At the start: 101 parts

Commit message: complete layout
Parts:
- removed LED100, LED101, LED83, LED84, LED85, LED86, LED87, LED88, LED89, LED90, LED91, LED92, LED93, LED94, LED95, LED96, LED97, LED98, LED99: ~, persional_library:LED-SMD_L3.2-W2.8_YO-WS2812B-3528, symbol persional_library:YO-WS2812B-3528反贴

Commit message: complete desin
Parts:
- added LED83, LED84, LED85: ~, persional_library:LED-SMD_L3.2-W2.8_YO-WS2812B-3528, symbol persional_library:YO-WS2812B-3528反贴
Connections:
- net +5V: now also LED83.1 (VDD), LED84.1 (VDD), LED85.1 (VDD)
- net GND: now also LED83.3 (GND), LED84.3 (GND), LED85.3 (GND)
- net LED6: now also LED85.2 (DOUT); no longer LED72.2 (DOUT)
- new net: LED84.2 (DOUT), LED85.4 (DIN)
- new net: LED83.2 (DOUT), LED84.4 (DIN)
- new net: LED72.2 (DOUT), LED83.4 (DIN)
