File: Hardware/KeyBoard/MCU.kicad_sch (KiCad schematic)
At the start: 0 parts

Commit message: Completed the schematic drawing, started the PCB process, and updated the firmware to the helloword firmware.
Parts:
- added C10, C11, C12, C13, C6, C7, C9: 100nF, persional_library:C0402, symbol persional_library:0402C
- added C4, C5, C8: 10uF, persional_library:C0402, symbol persional_library:0402C
- added CN1: ~, persional_library:CONN-TH_3P-P1.25_GH1.25, symbol persional_library:WAFER-GH1.25-3PWB
- added FPC2, FPC3: ~, persional_library:FPC-SMD_P0.50-8P_FGS-XJ-H2.0, symbol persional_library:FPC-8Pin
- added R24: 10kΩ, persional_library:R0402, symbol persional_library:0402R
- added R25, R26: 22Ω, persional_library:R0402, symbol persional_library:0402R
- added R27: 1.5kΩ, persional_library:R0402, symbol persional_library:0402R
- added SW1: ~, persional_library:SW-SMD_L6.0-W3.3-LS8.0, symbol persional_library:TS-1101-C-W
- added U13: ~, persional_library:LQFP-48_L7.0-W7.0-P0.50-LS9.0-BL, symbol persional_library:STM32F103CBT6
- added U14: ~, persional_library:SOT-25_L3.0-W1.6-P0.95-LS2.8-BL, symbol persional_library:XC6210B332MR_LDO3V3
- added X1: 8MHz, persional_library:OSC-SMD_3P-L3.2-W1.3-P1.20, symbol persional_library:CSTNE8M00GH5C000R0-8MHz
Connections:
- new net +3V3: C10.1, C11.1, C12.1, C13.1, C5.1, C6.1, C8.1, C9.1, R24.2, R27.2, U13.1 (VBAT), U13.24 (VDD_1), U13.36 (VDD_2), U13.48 (VDD_3), U13.9 (VDD_A), U14.5 (VOUT)
- new net +5V: C4.1, FPC2.7, FPC2.8, FPC3.7, FPC3.8, U14.1 (VIN), U14.3 (CE)
- new net CE: U13.39 (PB3JTDO)
- new net GND: C10.2, C11.2, C12.2, C13.2, C4.2, C5.2, C6.2, C7.2, C8.2, C9.2, CN1.3, CN1.4, CN1.5, FPC2.10, FPC2.5, FPC2.6, FPC2.9, FPC3.10, FPC3.5, FPC3.6, FPC3.9, SW1.2, U13.23 (VSS_1), U13.35 (VSS_2), U13.44 (BOOT0), U13.47 (VSS_3), U13.8 (VSS_A), U14.2 (VSS), X1.2 (GND)
- new net I2C1_SCL: FPC3.2, U13.42 (PB6I2C1_SCLTIM4_CH1)
- new net I2C1_SDA: FPC3.1, U13.43 (PB7I2C1_SDATIM4_CH2)
- new net I2C2_SCL: FPC3.3, U13.21 (PB10I2C2_SCLUSART3_TX)
- new net I2C2_SDA: FPC3.4, U13.22 (PB11I2C2_SDAUSART3_RX-)
- new net LED_CE: U13.28 (PB15SPI2_MOSITIM1_CH3N)
- new net NRST: C7.1, R24.1, SW1.1, U13.7 (NRST)
- new net OSC_IN: U13.5 (PD0-OSC_IN), X1.1 (OSC1)
- new net OSC_OUT: U13.6 (PD1-OSC_OUT), X1.3 (OSC2)
- new net PL: U13.40 (PB4NJTRST)
- new net SPI1_CLK: U13.15 (PA5SPI1_SCKADC12_IN5)
- new net SPI1_MISO: U13.16 (PA6SPI1_MISOADC12_IN6TIM3_CH1)
- new net SPI2_SCK: U13.26 (PB13SPI2_SCKUSART3_CTSTIM1_CH1N)
- new net SWCLK: CN1.1, U13.37 (PA14JTCKSWCLK)
- new net SWDIO: CN1.2, U13.34 (PA13JTMSSWDIO)
- new net UART_RX: FPC2.1, U13.31 (PA10USART1_RXTIM1_CH3)
- new net UART_TX: FPC2.2, U13.30 (PA9USART1_TXTIM1_CH2)
- new net USB_D_N: R25.1, U13.32 (PA11USART1_CTSCAN_RXTIM1_CH4USBDM)
- new net USB_D_P: R26.1, U13.33 (PA12USART1_RTSCAN_TXTIM1_ETRUSBDP)
- new net USB_PORT_N: FPC2.4, R25.2
- new net USB_PORT_P: FPC2.3, R26.2, R27.1
- no-connect marks 0 -> 20

Commit message: complete layout
Parts:
- removed FPC2: ~, persional_library:FPC-SMD_P0.50-8P_FGS-XJ-H2.0, symbol persional_library:FPC-8Pin
- removed SW1: ~, persional_library:SW-SMD_L6.0-W3.3-LS8.0, symbol persional_library:TS-1101-C-W
- added R28, R29: 10KΩ, persional_library:R0402, symbol persional_library:0402R
Connections:
- net GND: now also R28.2, R29.2; no longer U13.44 (BOOT0)
- net at U13.20 (PB2BOOT1): now also R29.1
- new net: R28.1, U13.44 (BOOT0)
- no-connect marks 20 -> 19

Commit message: start generic cabling
Connections:
- net SWCLK: now also CN1.2; no longer CN1.1
- net SWDIO: now also CN1.1; no longer CN1.2
Changed lines of the file:
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@@
+	(wire
+		(pts
+			(xy 60.96 105.41) (xy 66.04 105.41)
+		)
+		(stroke
+			(width 0)
+			(type default)
+		)
+	)
+	(wire
+		(pts
+			(xy 199.39 113.03) (xy 207.01 113.03)
+		)
+		(stroke
+			(width 0)
+			(type default)
+		)
+	)
+	(wire
+		(pts
+			(xy 146.05 138.43) (xy 146.05 143.51)
+		)
+		(stroke
+			(width 0)
+			(type default)
+		)
+	)
+	(wire
+		(pts
+			(xy 66.04 105.41) (xy 71.12 105.41)
+		)
+		(stroke
+			(width 0)
+			(type default)
+		)
+	)
+	(wire
+		(pts
+			(xy 58.42 128.27) (xy 59.69 128.27)
+		)
+		(stroke
+			(width 0)
+			(type default)
+		)
+	)
+	(wire
+		(pts
+			(xy 109.22 116.84) (xy 114.3 116.84)
+		)
+		(stroke
+			(width 0)
+			(type default)
+		)
+	)
+	(wire
+		(pts
+			(xy 199.39 118.11) (xy 207.01 118.11)
+		)
+		(stroke
+			(width 0)
+			(type default)
+		)
+	)
+	(wire
+		(pts
+			(xy 85.09 128.27) (xy 90.17 128.27)
+		)
+		(stroke
+			(width 0)
+			(type default)
+		)
+	)
+	(wire
+		(pts
+			(xy 146.05 129.54) (xy 152.4 129.54)
+		)
+		(stroke
+			(width 0)
+			(type default)
+		)
+	)
+	(wire
+		(pts
+			(xy 175.26 40.64) (xy 181.61 40.64)
+		)
+		(stroke
+			(width 0)
+			(type default)
+		)
+	)
+	(wire
+		(pts
+			(xy 87.63 151.13) (xy 93.98 151.13)
+		)
+		(stroke
+			(width 0)
+			(type default)
+		)
+	)
+	(wire
+		(pts
+			(xy 58.42 130.81) (xy 60.96 130.81)
+		)
+		(stroke
+			(width 0)
+			(type default)
+		)
+	)
+	(wire
+		(pts
+			(xy 175.26 73.66) (xy 181.61 73.66)
+		)
+		(stroke
+			(width 0)
+			(type default)
+		)
+	)
+	(wire
+		(pts
+			(xy 175.26 43.18) (xy 181.61 43.18)
+		)
+		(stroke
+			(width 0)
+			(type default)
+		)
+	)
+	(wire
+		(pts
+			(xy 57.15 55.88) (xy 62.23 55.88)
+		)
+		(stroke
+			(width 0)
+			(type default)
+		)
+	)
+	(wire
+		(pts
+			(xy 59.69 128.27) (xy 60.96 128.27)
+		)
+		(stroke
+			(width 0)
+			(type default)
+		)
+	)
+	(wire
+		(pts
+			(xy 62.23 38.1) (xy 68.58 38.1)
+		)
+		(stroke
+			(width 0)
+			(type default)
+		)
+	)
+	(wire
+		(pts
+			(xy 71.12 97.79) (xy 76.2 97.79)
+		)
+		(stroke
+			(width 0)
+			(type default)
+		)
+	)
 	(wire
 		(pts
@@
 	(wire
 		(pts
-			(xy 60.96 105.41) (xy 66.04 105.41)
-		)
-		(stroke
-			(width 0)
-			(type default)
-		)
-	)
-	(wire
-		(pts
-			(xy 199.39 113.03) (xy 207.01 113.03)
-		)
-		(stroke
-			(width 0)
-			(type default)
-		)
-	)
-	(wire
-		(pts
-			(xy 146.05 138.43) (xy 146.05 143.51)
-		)
-		(stroke
-			(width 0)
-			(type default)
-		)
-	)
-	(wire
-		(pts
-			(xy 66.04 105.41) (xy 71.12 105.41)
-		)
-		(stroke
-			(width 0)
-			(type default)
-		)
-	)
-	(wire
-		(pts
-			(xy 58.42 128.27) (xy 59.69 128.27)
-		)
-		(stroke
-			(width 0)
-			(type default)
-		)
-	)
-	(wire
-		(pts
-			(xy 109.22 116.84) (xy 114.3 116.84)
-		)
-		(stroke
-			(width 0)
-			(type default)
-		)
-	)
-	(wire
-		(pts
-			(xy 199.39 118.11) (xy 207.01 118.11)
-		)
-		(stroke
-			(width 0)
-			(type default)
-		)
-	)
-	(wire
-		(pts
-			(xy 85.09 128.27) (xy 90.17 128.27)
-		)
-		(stroke
-			(width 0)
-			(type default)
-		)
-	)
-	(wire
-		(pts
-			(xy 146.05 129.54) (xy 152.4 129.54)
-		)
-		(stroke
-			(width 0)
-			(type default)
-		)
-	)
-	(wire
-		(pts
-			(xy 175.26 40.64) (xy 181.61 40.64)
-		)
-		(stroke
-			(width 0)
-			(type default)
-		)
-	)
-	(wire
-		(pts
-			(xy 87.63 151.13) (xy 93.98 151.13)
-		)
-		(stroke
-			(width 0)
-			(type default)
-		)
-	)
-	(wire
-		(pts
-			(xy 58.42 130.81) (xy 60.96 130.81)
-		)
-		(stroke
-			(width 0)
-			(type default)
-		)
-	)
-	(wire
-		(pts
-			(xy 175.26 73.66) (xy 181.61 73.66)
-		)
-		(stroke
-			(width 0)
-			(type default)
-		)
-	)
-	(wire
-		(pts
-			(xy 175.26 43.18) (xy 181.61 43.18)
-		)
-		(stroke
-			(width 0)
-			(type default)
-		)
-	)
-	(wire
-		(pts
-			(xy 57.15 55.88) (xy 62.23 55.88)
-		)
-		(stroke
-			(width 0)
-			(type default)
-		)
-	)
-	(wire
-		(pts
-			(xy 59.69 128.27) (xy 60.96 128.27)
-		)
-		(stroke
-			(width 0)
-			(type default)
-		)
-	)
-	(wire
-		(pts
-			(xy 62.23 38.1) (xy 68.58 38.1)
-		)
-		(stroke
-			(width 0)
-			(type default)
-		)
-	)
-	(wire
-		(pts
-			(xy 71.12 97.79) (xy 76.2 97.79)
-		)
-		(stroke
-			(width 0)
-			(type default)
-		)
-	)
-	(wire
-		(pts
 			(xy 175.26 83.82) (xy 181.61 83.82)
 		)
@@
 	(wire
 		(pts
+			(xy 265.43 118.11) (xy 270.51 118.11)
+		)
+		(stroke
+			(width 0)
+			(type default)
+		)
+	)
+	(wire
+		(pts
 			(xy 175.26 68.58) (xy 181.61 68.58)
 		)
@@
 	(wire
 		(pts
-			(xy 265.43 118.11) (xy 270.51 118.11)
-		)
-		(stroke
-			(width 0)
-			(type default)
-		)
-	)
-	(wire
-		(pts
 			(xy 104.14 151.13) (xy 113.03 151.13)
 		)
@@
 			(width 0)
 			(type default)
+		)
+	)
+	(label "SWCLK"
+		(at 265.43 118.11 0)
+		(effects
+			(font
+				(size 1.27 1.27)
+			)
+			(justify left bottom)
 		)
 	)
@@
 		)
 	)
-	(label "SWDIO"
-		(at 265.43 118.11 0)
-		(effects
-			(font
-				(size 1.27 1.27)
-			)
-			(justify left bottom)
-		)
-	)
 	(label "NRST"
 		(at 68.58 43.18 180)
@@
 		)
 	)
+	(label "SWDIO"
+		(at 265.43 115.57 0)
+		(effects
+			(font
+				(size 1.27 1.27)
+			)
+			(justify left bottom)
+		)
+	)
 	(label "OSC_IN"
 		(at 124.46 116.84 0)
@@
 		(effects
 			(font
-				(size 1.27 1.27)
-			)
-			(justify left bottom)
-		)
-	)
-	(label "SWCLK"
-		(at 265.43 115.57 0)
-		(effects
-			(font

Commit message: complete desin
Changed lines of the file:
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@@
 					(size 1.27 1.27)
 				)
-				(hide yes)
 			)
 		)
